File: hardware/motor_driver/motor_driver.sch (EAGLE design)
At the start: 38 parts

Commit message: Made changes
Parts:
- added C6: 6.8nF, adafruit:C-USC0603
- added C7: 120pF, adafruit:C-USC0603
- added C8: 22nF, adafruit:C-USC0603
- added R20: 15K, adafruit:R-US_R0603
- added R21: 220K, adafruit:R-US_R0603
- added R22, R24: (no value), adafruit:R-US_R0603
- added R23: 10K, adafruit:R-US_R0603
- added R25: 0R, adafruit:R-US_R0603
Connections:
- net SOMEOTHERGND renamed AGND
- new net N$10: C8.1, U$7.CP1
- new net N$13: C8.2, U$7.CP2
- new net N$14: C7.1, R20.1
- new net N$15: R21.2, U$7.RT_CLK
- new net N$17: R25.2, U$7.EN_BUCK
- new net N$20: C6.1, R20.2, U$7.COMP
- new net PWRGD: R23.2, U$7.PWRGD
- net +5V: now also R23.1
- net DGND: now also C6.2, C7.2, R21.1, R25.1
Other:
- note added: "Connect to GND with a very short trace."
- note added: "R21 is external clock for buck converter."
Changed lines of the file:
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@@
 <part name="R19" library="adafruit" deviceset="R-US_" device="R0603" value="10M"/>
 <part name="SUPPLY8" library="supply2" deviceset="DGND" device=""/>
+<part name="R20" library="adafruit" deviceset="R-US_" device="R0603" value="15K"/>
+<part name="R21" library="adafruit" deviceset="R-US_" device="R0603" value="220K"/>
+<part name="R22" library="adafruit" deviceset="R-US_" device="R0603"/>
+<part name="R23" library="adafruit" deviceset="R-US_" device="R0603" value="10K"/>
+<part name="R24" library="adafruit" deviceset="R-US_" device="R0603"/>
+<part name="C6" library="adafruit" deviceset="C-US" device="C0603" value="6.8nF"/>
+<part name="C7" library="adafruit" deviceset="C-US" device="C0603" value="120pF"/>
+<part name="C8" library="adafruit" deviceset="C-US" device="C0603" value="22nF"/>
+<part name="SUPPLY9" library="supply2" deviceset="DGND" device=""/>
+<part name="P+6" library="supply1" deviceset="+5V" device=""/>
+<part name="R25" library="adafruit" deviceset="R-US_" device="R0603" value="0R"/>
+<part name="SUPPLY10" library="supply2" deviceset="DGND" device=""/>
 </parts>
 <sheets>
@@
 <text x="190.5" y="7.62" size="0.6096" layer="97">Ioc = (R18/ (R17+R18) * 3.3[DVDD] ) / Rds(on)</text>
 <text x="241.3" y="10.16" size="0.6096" layer="97">90 A Cutoff</text>
+<text x="193.04" y="-63.5" size="0.508" layer="97" rot="R90">R21 is external clock for buck converter.</text>
+<text x="194.31" y="-63.5" size="0.508" layer="97" rot="R90"> Connect to GND with a very short trace.</text>
 </plain>
 <instances>
@@
 <instance part="R19" gate="G$1" x="218.44" y="7.62"/>
 <instance part="SUPPLY8" gate="G$1" x="210.82" y="5.08"/>
+<instance part="R20" gate="G$1" x="205.74" y="-50.8" rot="R90"/>
+<instance part="R21" gate="G$1" x="198.12" y="-53.34" rot="R90"/>
+<instance part="R22" gate="G$1" x="182.88" y="-38.1" rot="R90"/>
+<instance part="R23" gate="G$1" x="215.9" y="-38.1"/>
+<instance part="R24" gate="G$1" x="175.26" y="-53.34" rot="R90"/>
+<instance part="C6" gate="G$1" x="213.36" y="-53.34"/>
+<instance part="C7" gate="G$1" x="205.74" y="-58.42"/>
+<instance part="C8" gate="G$1" x="223.52" y="-60.96" rot="R90"/>
+<instance part="SUPPLY9" gate="G$1" x="205.74" y="-66.04"/>
+<instance part="P+6" gate="1" x="205.74" y="-38.1" rot="R90"/>
+<instance part="R25" gate="G$1" x="205.74" y="-35.56"/>
+<instance part="SUPPLY10" gate="G$1" x="198.12" y="-35.56" rot="R270"/>
 </instances>
 <busses>
@@
 </segment>
 </net>
-<net name="SOMEOTHERGND" class="0">
+<net name="AGND" class="0">
 <segment>
 <pinref part="CURR" gate="-5" pin="S"/>
@@
 <pinref part="SUPPLY8" gate="G$1" pin="DGND"/>
 <wire x1="210.82" y1="7.62" x2="213.36" y2="7.62" width="0.1524" layer="91"/>
+</segment>
+<segment>
+<pinref part="C6" gate="G$1" pin="2"/>
+<wire x1="213.36" y1="-58.42" x2="213.36" y2="-63.5" width="0.1524" layer="91"/>
+<pinref part="C7" gate="G$1" pin="2"/>
+<wire x1="213.36" y1="-63.5" x2="205.74" y2="-63.5" width="0.1524" layer="91"/>
+<pinref part="R21" gate="G$1" pin="1"/>
+<wire x1="198.12" y1="-58.42" x2="198.12" y2="-63.5" width="0.1524" layer="91"/>
+<wire x1="198.12" y1="-63.5" x2="205.74" y2="-63.5" width="0.1524" layer="91"/>
+<junction x="205.74" y="-63.5"/>
+<pinref part="SUPPLY9" gate="G$1" pin="DGND"/>
+</segment>
+<segment>
+<pinref part="R25" gate="G$1" pin="1"/>
+<pinref part="SUPPLY10" gate="G$1" pin="DGND"/>
 </segment>
 </net>
@@
 <junction x="218.44" y="40.64"/>
 </segment>
+<segment>
+<pinref part="R23" gate="G$1" pin="1"/>
+<pinref part="P+6" gate="1" pin="+5V"/>
+<wire x1="208.28" y1="-38.1" x2="210.82" y2="-38.1" width="0.1524" layer="91"/>
+</segment>
 </net>
 <net name="M_PWM" class="0">
@@
 </segment>
 </net>
+<net name="N$10" class="0">
+<segment>
+<pinref part="U$7" gate="G$1" pin="CP1"/>
+<pinref part="C8" gate="G$1" pin="1"/>
+<wire x1="226.06" y1="-48.26" x2="220.98" y2="-48.26" width="0.1524" layer="91"/>
+<wire x1="220.98" y1="-48.26" x2="220.98" y2="-60.96" width="0.1524" layer="91"/>
+</segment>
+</net>
+<net name="N$13" class="0">
+<segment>
+<pinref part="U$7" gate="G$1" pin="CP2"/>
+<wire x1="226.06" y1="-50.8" x2="226.06" y2="-53.34" width="0.1524" layer="91"/>
+<pinref part="C8" gate="G$1" pin="2"/>
+<wire x1="226.06" y1="-53.34" x2="228.6" y2="-53.34" width="0.1524" layer="91"/>
+<wire x1="228.6" y1="-53.34" x2="228.6" y2="-60.96" width="0.1524" layer="91"/>
+</segment>
+</net>
+<net name="N$14" class="0">
+<segment>
+<pinref part="C7" gate="G$1" pin="1"/>
+<pinref part="R20" gate="G$1" pin="1"/>
+</segment>
+</net>
+<net name="N$20" class="0">
+<segment>
+<pinref part="R20" gate="G$1" pin="2"/>
+<pinref part="U$7" gate="G$1" pin="COMP"/>
+<wire x1="226.06" y1="-45.72" x2="213.36" y2="-45.72" width="0.1524" layer="91"/>
+<pinref part="C6" gate="G$1" pin="1"/>
+<wire x1="213.36" y1="-45.72" x2="205.74" y2="-45.72" width="0.1524" layer="91"/>
+<wire x1="213.36" y1="-50.8" x2="213.36" y2="-45.72" width="0.1524" layer="91"/>
+<junction x="213.36" y="-45.72"/>
+</segment>
+</net>
+<net name="N$15" class="0">
+<segment>
+<pinref part="R21" gate="G$1" pin="2"/>
+<pinref part="U$7" gate="G$1" pin="RT_CLK"/>
+<wire x1="226.06" y1="-43.18" x2="198.12" y2="-43.18" width="0.1524" layer="91"/>
+<wire x1="198.12" y1="-43.18" x2="198.12" y2="-48.26" width="0.1524" layer="91"/>
+</segment>
+</net>
+<net name="PWRGD" class="0">
+<segment>
+<pinref part="R23" gate="G$1" pin="2"/>
+<pinref part="U$7" gate="G$1" pin="PWRGD"/>
+<wire x1="220.98" y1="-38.1" x2="226.06" y2="-38.1" width="0.1524" layer="91"/>
+<label x="220.98" y="-38.1" size="0.508" layer="95" rot="R270" xref="yes"/>
+</segment>
+</net>
+<net name="N$17" class="0">
+<segment>
+<pinref part="R25" gate="G$1" pin="2"/>
+<pinref part="U$7" gate="G$1" pin="EN_BUCK"/>
+<wire x1="210.82" y1="-35.56" x2="226.06" y2="-35.56" width="0.1524" layer="91"/>
+</segment>
+</net>

Commit message: Completed first revision of design
Parts:
- added C10: 100nF, SparkFun-Passives:CAP0805
- added C11, C12, C13, C14, C19, C20, C21, C23: 10u,50V, SparkFun-Passives:CAP1206
- added C15, C16, C17, C18, C25: 2.2u, adafruit:C-USC0805
- added C22, C24: 15u,100V, resistor:C-EUC2220K
- added C26, C9: 100uF, SparkFun-Capacitors:CAP_POL3528-KIT
- added CTRL, SENS: 22-23-2041, con-molex:22-23-2041
- added D1: PMEG6020ER,115, nxp:DIODE[SCHOTKY]-SOD123W
- added D2: SMAJ5.0A, SparkFun-DiscreteSemi:TVSSMA
- added L1: 22uH, bourne:SDR0805
- added PT1, PT2: 2PT_GND_TIE, SparkFun-Passives:2PT_GND_TIE
- added R26, R28, R30: 39K, adafruit:R-US_R0805
- added R27, R29, R31: 2.2K, adafruit:R-US_R0805
- added U$10: TC2117, bldc_lib:TC2117
- JP2: value (none) -> M_PWM
- JP3: value (none) -> M_OC
- JP4: value (none) -> GAIN
- R22: value (none) -> 3.3K
- R24: value (none) -> 18K
Connections:
- removed net V_SUPPLY: U$1.D, U$4.D, U$5.D
- new net +3V3: C25.1, C26.+, U$10.VOUT
- new net N$18: C15.1, U$7.GVDD
- new net N$19: C10.2, D1.2, L1.2, U$7.PH1, U$7.PH2
- new net N$27: C16.1, U$7.AVDD
- new net N$28: R22.2, R24.1, U$7.VSENSE
- new net N$29: C10.1, U$7.BST_BK
- new net N$30: C17.1, C18.1, U$7.DVDD
- new net SENS1: R26.2, R27.2, SENS-3.S
- new net SENS2: R28.2, R29.2, SENS-2.S
- new net SENS3: R30.2, R31.2, SENS-1.S
- new net VCC: C11.2, C12.1, C13.1, C14.1, C19.2, C20.2, C21.2, C22.2, C23.2, C24.2, U$1.D, U$4.D, U$5.D, U$7.PVDD1, U$7.PVDD2, U$7.PVDD2(2)
- net +5V: now also C9.+, D2.C, L1.1, R24.2, U$10.VI
- net AGND: now also C16.2, C17.2, C18.2, PT2.P$2, R27.1, R29.1, R31.1, SENS-4.S, U$7.AGND
- net DGND: now also C25.2, C26.-, C9.-, CTRL-4.S, D1.1, D2.A, PT1.P$2, R22.1, U$10.GND
- net FAULT: now also CTRL-2.S
- net GND: now also C11.1, C12.2, C13.2, C14.2, C15.2, C19.1, C20.1, C21.1, C22.1, C23.1, C24.1, PT1.P$1, PT2.P$1, U$7.GND
- net H1_VS: now also R26.1
- net H2_VS: now also R28.1
- net H3_VS: now also R30.1
- net OCTW: now also CTRL-3.S
- net PWRGD: now also CTRL-1.S
Other:
- note added: "1.0"
- note added: "3.3V Regulator for logic"
- note added: "A TVS diode, or transient voltage suppression diode, is an electrical device which is designed to divert or shunt voltage spikes from a circuit in order to protect that circuit."
- note added: "BUCK REGULATOR CIRCUIT"
- note added: "Connect Grounds"
- note added: "Control Connector"
- note added: "DRIVER"
- note added: "Don't mount R18, because internal current limit of DRV8302 doesn't work with this config for some reason"
- note added: "Motor Driver (2015)"
- note added: "Rumman Waqar; Mike Bardwell"
- note added: "SDR0805-220ML"
- note added: "Sense Voltage at each phase"
- note added: "TPSB107K006R0400"
- note added: "Voltage Smoothing"
- moved on the sheet: JP2, JP3, JP4, R1, R2, R22, R24, R3, R4, R5, R6, R7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
